File: tf_chess.kicad_pcb (KiCad board)
At the start: 2 copper layers, 456 x 456 mm, 0 parts

Commit message: initial release
Other:
- outline, holes or cut-outs redrawn
- board text added: "2025-10-05"
- board text added: "M. House"
Changed lines of the file:
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@@
 			(drillshape 0)
 			(scaleselection 1)
-			(outputdirectory "v2")
+			(outputdirectory "v3/")
 		)
 	)
@@
 		(layer "B.Mask")
 	)
-	(gr_rect
-		(start -49.5 -104)
-		(end 406.5 352)
+	(gr_arc
+		(start 406.5 347)
+		(mid 405.035534 350.535534)
+		(end 401.5 352)
 		(stroke
 			(width 0.1)
 			(type solid)
 		)
-		(fill no)
+		(layer "Edge.Cuts")
+	)
+	(gr_line
+		(start -49.5 347)
+		(end -49.5 -99)
+		(stroke
+			(width 0.1)
+			(type solid)
+		)
+		(layer "Edge.Cuts")
+	)
+	(gr_arc
+		(start -49.5 -99)
+		(mid -48.035534 -102.535534)
+		(end -44.5 -104)
+		(stroke
+			(width 0.1)
+			(type solid)
+		)
+		(layer "Edge.Cuts")
+	)
+	(gr_line
+		(start 406.5 -99)
+		(end 406.5 347)
+		(stroke
+			(width 0.1)
+			(type solid)
+		)
+		(layer "Edge.Cuts")
+	)
+	(gr_line
+		(start -44.5 -104)
+		(end 401.5 -104)
+		(stroke
+			(width 0.1)
+			(type solid)
+		)
+		(layer "Edge.Cuts")
+	)
+	(gr_arc
+		(start -44.5 352)
+		(mid -48.035534 350.535534)
+		(end -49.5 347)
+		(stroke
+			(width 0.1)
+			(type solid)
+		)
+		(layer "Edge.Cuts")
+	)
+	(gr_arc
+		(start 401.5 -104)
+		(mid 405.035534 -102.535534)
+		(end 406.5 -99)
+		(stroke
+			(width 0.1)
+			(type solid)
+		)
+		(layer "Edge.Cuts")
+	)
+	(gr_line
+		(start 401.5 352)
+		(end -44.5 352)
+		(stroke
+			(width 0.1)
+			(type solid)
+		)
 		(layer "Edge.Cuts")
 	)
@@
 		)
 	)
+	(gr_text "M. House"
+		(at 378 314 0)
+		(layer "F.Cu")
+		(effects
+			(font
+				(size 6 6)
+				(thickness 1.1)
+			)
+		)
+	)
 	(gr_text "A4"
 		(at -37.5 172 0)
@@
 			)
 		)
+	)
+	(gr_text "2025-10-05"
+		(at 378 328 0)
+		(layer "F.Cu")
+		(effects
+			(font
+				(size 5 5)
+				(thickness 0.9)
+			)
+		)
